File: P1P2 Adapter.sch (KiCad schematic (older format))
At the start: 31 parts, among them J1 Conn_01x07_Male, J2 Conn_01x01_Male, J3 Conn_01x01_Male, U1 MAX22088

Commit message: Updated ground plane and PCB design
Connections:
- net GND: now also U1.25 (GND)
Changed lines of the file:
@@
 	6350 3900 6350 4000
 Connection ~ 6350 4000
+$Comp
+L power:GND #PWR019
+U 1 1 6141948B
+P 6200 4650
+F 0 "#PWR019" H 6200 4400 50  0001 C CNN
+F 1 "GND" H 6205 4477 50  0000 C CNN
+F 2 "" H 6200 4650 50  0001 C CNN
+F 3 "" H 6200 4650 50  0001 C CNN
+	1    6200 4650
+	1    0    0    -1
+$EndComp
 $EndSCHEMATC

Commit message: Fixed incorrect trim resistors and termination resistors. Credit goes to Arnold N, creator of P1P2Serial
Parts:
- R10: value 168k -> 20k
- R4: value 100 -> 1k
- R5: value 100 -> 82
- R8: value 1M -> 27k
- R9: value 220k -> 4.3k
Connections:
- net TVL: now also R8.2, R9.1; no longer R10.1, R9.2
- net TVT: now also R10.1, R9.2; no longer R8.2, R9.1
Changed lines of the file:
@@
 P 4500 5750
 F 0 "R5" H 4570 5796 50  0000 L CNN
-F 1 "100" H 4570 5705 50  0000 L CNN
+F 1 "82" H 4570 5705 50  0000 L CNN
 F 2 "Resistor_SMD:R_1206_3216Metric_Pad1.30x1.75mm_HandSolder" V 4430 5750 50  0001 C CNN
 F 3 "~" H 4500 5750 50  0001 C CNN
@@
 P 4500 5100
 F 0 "R4" H 4570 5146 50  0000 L CNN
-F 1 "100" H 4570 5055 50  0000 L CNN
+F 1 "1k" H 4570 5055 50  0000 L CNN
 F 2 "Resistor_SMD:R_1206_3216Metric_Pad1.30x1.75mm_HandSolder" V 4430 5100 50  0001 C CNN
 F 3 "~" H 4500 5100 50  0001 C CNN
@@
 TVL
 Text GLabel 7450 3250 2    50   Output ~ 0
+TVL
+Text GLabel 7450 3550 2    50   Output ~ 0
 TVT
-Text GLabel 7450 3550 2    50   Output ~ 0
-TVL
 $Comp
 L power:+5V #PWR09
@@
 P 7300 3100
 F 0 "R8" H 7370 3146 50  0000 L CNN
-F 1 "1M" H 7370 3055 50  0000 L CNN
+F 1 "27k" H 7370 3055 50  0000 L CNN
 F 2 "Resistor_SMD:R_1206_3216Metric_Pad1.30x1.75mm_HandSolder" V 7230 3100 50  0001 C CNN
 F 3 "~" H 7300 3100 50  0001 C CNN
@@
 P 7300 3400
 F 0 "R9" H 7370 3446 50  0000 L CNN
-F 1 "220k" H 7370 3355 50  0000 L CNN
+F 1 "4.3k" H 7370 3355 50  0000 L CNN
 F 2 "Resistor_SMD:R_1206_3216Metric_Pad1.30x1.75mm_HandSolder" V 7230 3400 50  0001 C CNN
 F 3 "~" H 7300 3400 50  0001 C CNN
@@
 P 7300 3700
 F 0 "R10" H 7370 3746 50  0000 L CNN
-F 1 "168k" H 7370 3655 50  0000 L CNN
+F 1 "20k" H 7370 3655 50  0000 L CNN
 F 2 "Resistor_SMD:R_1206_3216Metric_Pad1.30x1.75mm_HandSolder" V 7230 3700 50  0001 C CNN
 F 3 "~" H 7300 3700 50  0001 C CNN

Commit message: Made changes for 9600bps operation
Parts:
- C1, C2: value 1u -> 22u
- R4: value 1k -> 240
Changed lines of the file:
@@
 P 4500 5100
 F 0 "R4" H 4570 5146 50  0000 L CNN
-F 1 "1k" H 4570 5055 50  0000 L CNN
+F 1 "240" H 4570 5055 50  0000 L CNN
 F 2 "Resistor_SMD:R_1206_3216Metric_Pad1.30x1.75mm_HandSolder" V 4430 5100 50  0001 C CNN
 F 3 "~" H 4500 5100 50  0001 C CNN
@@
 P 3450 4700
 F 0 "C1" V 3702 4700 50  0000 C CNN
-F 1 "1u" V 3611 4700 50  0000 C CNN
+F 1 "22u" V 3611 4700 50  0000 C CNN
 F 2 "Capacitor_SMD:C_1206_3216Metric_Pad1.33x1.80mm_HandSolder" H 3488 4550 50  0001 C CNN
 F 3 "~" H 3450 4700 50  0001 C CNN
@@
 P 3450 5500
 F 0 "C2" V 3702 5500 50  0000 C CNN
-F 1 "1u" V 3611 5500 50  0000 C CNN
+F 1 "22u" V 3611 5500 50  0000 C CNN
 F 2 "Capacitor_SMD:C_1206_3216Metric_Pad1.33x1.80mm_HandSolder" H 3488 5350 50  0001 C CNN
 F 3 "~" H 3450 5500 50  0001 C CNN
